Commit message: Actualizamos el Robot virtual.

File: Fase_1/Nodo_ROS2/RViz/roomba.urdf (robot description, URDF)
Before this commit: robot roomba, 2 links, 1 joints
Links:
- removed link wheel
- added link base_footprint
- added link caster_wheel, mass 0.1; collision sphere radius=0.025; visual sphere radius=0.025
- added link left_wheel; collision cylinder length=0.03 radius=0.035; visual cylinder length=0.03 radius=0.035
- added link right_wheel; collision cylinder length=0.03 radius=0.035; visual cylinder length=0.03 radius=0.035
- link base_link: mass None -> 2.5; geometry collision cylinder length=0.1 radius=0.17; visual cylinder length=0.1 radius=0.17
Joints:
- removed joint base_to_wheel
- added joint base_joint: type fixed, parent base_footprint, child base_link, origin xyz=0 0 0.05 rpy=0 0 0
- added joint caster_joint: type fixed, parent base_link, child caster_wheel, origin xyz=0.12 0 -0.05 rpy=0 0 0
- added joint left_wheel_joint: type continuous, parent base_link, child left_wheel, origin xyz=0 0.15 -0.025 rpy=-1.5708 0 0, axis 0 0 1
- added joint right_wheel_joint: type continuous, parent base_link, child right_wheel, origin xyz=0 -0.15 -0.025 rpy=-1.5708 0 0, axis 0 0 1
